File: ESP32-S3-GPS.kicad_sch (KiCad schematic)
At the start: 46 parts, among them J1 PJ-102, J10 Conn_01x04_Pin, J11 Conn_01x04, J12 Conn_01x04, J2 Conn_01x03, J3 Conn_01x04, J4 Conn_01x05, J5 USB_B_Mini, J6 Conn_01x03_Pin, J7 Conn_01x02_Pin, J8 Conn_01x02_Pin, J9 Conn_02x04_Odd_Even, U1 AMS1117-5.0, U2 CH340N, U3 AMS1117-3.3, U5 ESP32-S3-DEVKITC-1-N8R2, U6 NRF24L01_Breakout

Commit message: Change width of ESP32 Module footprint.  Change debug pin.
Connections:
- net Dbg1: now also U5.J3_16 (GPIO48); no longer U5.J3_15 (GPIO45)
- net SDA: now also U5.J3_15 (GPIO45); no longer U5.J3_16 (GPIO48)
Changed lines of the file:
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@@
 	)
 	(label "SDA"
-		(at 231.14 72.39 180)
+		(at 231.14 69.85 180)
 		(effects
 			(font
@@
 	)
 	(label "Dbg1"
-		(at 231.14 69.85 180)
-		(effects
-			(font
+		(at 231.14 72.39 180)
+		(effects
+			(font
